File: kicad/uRX/uRX.kicad_sch (KiCad schematic)
At the start: 109 parts, among them J1 RF_GMD, J2 C165948, J3 AudioJack2_Ground, J4 +5Vfiltered, J5 +5V, J6 U.FL, J7 +3.3Vfiltered, J9 RF_In, Q1 BC847, SW1 RotaryEncoder_Switch, U1 CBT3253, U10 IP2326, U12 OPA2211, U2 LM4562, U3 ESP32-DEVKIT, U4 Si5351A-B-GT, U6 Si4732-A10, U7 PCM1808PWR, U8 LM4040-2.5, U9 PCM1808PWR, Y1 25MHz, Y2 32768kHz

Commit message: add esp32 to pcb
Parts:
- removed R17, R7: 4.7kΩ, Resistor_SMD:R_0603_1608Metric, symbol Device:R_Small
- removed R21, R22, R23, R24: 22, Resistor_SMD:R_0603_1608Metric, symbol Device:R
- removed SW1: RotaryEncoder_Switch, RotaryEncoder_Alps_EC11E-Switch_Vertical_H20mm, symbol Device:RotaryEncoder_Switch
- removed U3: ESP32-DEVKIT, parts:MODULE_ESP32_DEVKIT_V1, symbol ESP32-DEVKIT-V1:ESP32-DEVKIT-V1
- added C24: 1u, Capacitor_SMD:C_0603_1608Metric, symbol uRX:C_Small
- added C25: 47u, Capacitor_SMD:C_0603_1608Metric, symbol uRX:C_Small
- added C32: 10n, Capacitor_SMD:C_0603_1608Metric, symbol uRX:C_Small
- added C33, C38, C39: 100n, Capacitor_SMD:C_0603_1608Metric, symbol uRX:C_Small
- added D2, D5: D_Schottky, D_SOD-123, symbol Device:D_Schottky
- added R13, R9: 4.7K, Resistor_SMD:R_0603_1608Metric, symbol Device:R_Small
- added R14, R15: 10k, Resistor_SMD:R_0603_1608Metric, symbol Device:R_Small
- added R16, R25, R29, R30: 22, Resistor_SMD:R_0603_1608Metric, symbol Device:R
- added SW2: RotaryEncoder_Switch, RotaryEncoder_Alps_EC11E-Switch_Vertical_H20mm, symbol Device:RotaryEncoder_Switch
- added SW3: Reset, SW_SPST_B3U-1000P, symbol Switch:SW_Push
- added SW4: Boot, SW_SPST_B3U-1000P, symbol Switch:SW_Push
- added U11: LP2985-5.0, Package_TO_SOT_SMD:SOT-23-5, symbol Regulator_Linear:LP2985-5.0
- added U13: HT733333, Package_TO_SOT_SMD:SOT-23-5, symbol Regulator_Linear:AP2112K-3.3
- added U5: ESP32-S3-WROOM-2, PCM_Espressif:ESP32-S3-WROOM-2, symbol PCM_Espressif:ESP32-S3-WROOM-2
- J1: value RF_GMD -> RF_AM_GND
- J6: footprint PCM_JLCPCB:IPEX-SMD_BWIPX-1-001E -> SMA_Molex_73251-1153_EdgeMount_Horizontal
- J9: value RF_In -> RF_AM__In
- U6: footprint Package_SO:SOIC-8_3.9x4.9mm_P1.27mm -> Package_SO:SSOP-16_3.9x4.9mm_P0.635mm
Connections:
- net +3.3V: now also C25.1, R13.1, R14.1, R15.1, R9.1, U13.5 (VOUT), U5.2 (3V3)
- net +5V: now also U11.5 (VOUT), U13.1 (VIN), U13.3 (EN); no longer Bat2.3 (Pin_3), Bat3.3 (Pin_3), U10.21 (VOUT), U10.22 (VOUT)
- net +5Vfiltered: no longer Bat2.1 (Pin_1), Bat3.1 (Pin_1), C10.2, C11.2, C13.2, C14.2, C19.1, C2.2, C20.1, C21.1, C22.1, C23.1, C26.2, C27.2, C28.1, C29.1, C3.2, C30.1, C31.1, C34.2, C36.2, C37.2, C4.2, C40.2, C41.2, C43.2, C5.2, C8.2, C9.2, D3.1 (K), D4.1 (K), D6.2 (A), J1.1 (Pin_1), J2.A1 (GND), J2.A12 (GND), J2.B1 (GND), J2.B12 (GND), J6.2 (Ext), Q1.2 (E), R34.2, R35.2, R36.2, R37.2, R41.2, R42.2, R43.2, R44.2, U1.1 (1~{OE}), U1.15 (2~{OE}), U1.8 (GND), U10.18 (PGND), U10.24 (VBAT_GND), U12.4 (V-), U4.8 (GND), U6.10 (SENB), U6.15 (GND), U7.10 (MD0), U7.11 (MD1), U7.12 (FMT), U7.2 (AGND), U7.5 (DGND), U8.5 (A), U9.10 (MD0), U9.11 (MD1), U9.12 (FMT), U9.2 (AGND), U9.5 (DGND)
- net I2S0_DOUT: now also U7.9 (DOUT), R16.1
- net I2S1_DOUT: now also U9.9 (DOUT), R25.1
- net SCL: now also R13.2, U5.17 (GPIO9/TOUCH9/ADC1_CH8/FSPIHD/SUBSPIHD)
- net SDA: now also R9.2, U5.12 (GPIO8/TOUCH8/ADC1_CH7/SUBSPICS1)
- net VBUS: now reaches C34.1, J2.A4 (VBUS), J2.A9 (VBUS), J2.B4 (VBUS), J2.B9 (VBUS), L2.2, R44.1, U10.12 (EN), U10.13 (VIN)
- net VBUS: now also D2.2 (A)
- net USB_D+: now reaches J2.A6 (D+), J2.B6 (D+)
- net USB_D+: now also R29.1; no longer U10.2 (DP)
- net USB_D-: now reaches J2.A7 (D-), J2.B7 (D-)
- net USB_D-: now also R30.1; no longer U10.1 (DM)
- net Q_BAT_STAT: now reaches Q1.3 (C)
- net Q_BAT_STAT: now also U5.39 (GPIO1/TOUCH1/ADC1_CH0)
- net RST_4732: now reaches R5.2, U6.9 (RST)
- net RST_4732: now also U5.7 (GPIO7/TOUCH7/ADC1_CH6)
- net I2S_BCK: now reaches U9.8 (BCK)
- net I2S_BCK: now also R1.1, U7.8 (BCK)
- net ADC_SCKI: now reaches Rf1.1, U7.6 (SCKI), U9.6 (SCKI)
- net ADC_SCKI: now also U5.18 (GPIO10/TOUCH10/ADC1_CH9/FSPICS0/FSPIIO4/SUBSPICS0)
- net I2S_LRCK: now reaches U7.7 (LRCK)
- net I2S_LRCK: now also R2.1, U9.7 (LRCK); no longer R1.1
- net I2S0_BCK: no longer names the net of R2.2
- net I2S0_BCK: now also U5.20 (GPIO12/TOUCH12/ADC2_CH1/FSPICLK/FSPIIO6/SUBSPICLK)
- net I2S0_LRCK: no longer names the net of R1.2
- net I2S0_LRCK: now also U5.19 (GPIO11/TOUCH11/ADC2_CH0/FSPID/FSPIIO5/SUBSPID)
- new net: D2.1 (K), D5.1 (K), U11.1 (VIN), U11.3 (ON/~{OFF})
- new net: C32.1, U11.4 (BP)
- new net: R15.2, SW4.1, U5.27 (GPIO0/BOOT)
- new net: R16.2, U5.21 (GPIO13/TOUCH13/ADC2_CH2/FSPIQ/FSPIIO7/SUBSPIQ)
- new net: C38.2, SW2.B, U5.5 (GPIO5/TOUCH5/ADC1_CH4)
- new net: R30.2, U5.13 (GPIO19/U1RTS/ADC2_CH8/CLK_OUT2/USB_D-)
- new net: R29.2, U5.14 (GPIO20/U1CTS/ADC2_CH9/CLK_OUT1/USB_D+)
- new net: R25.2, U5.22 (GPIO14/TOUCH14/ADC2_CH3/FSPIWP/FSPIDQS/SUBSPIWP)
- new net: C24.1, R14.2, SW3.2, U5.3 (EN)
- new net: C33.2, SW2.A, U5.4 (GPIO4/TOUCH4/ADC1_CH3)
- new net: C39.1, SW2.S1, U5.6 (GPIO6/TOUCH6/ADC1_CH5)
- new net +VBatt: Bat2.3 (Pin_3), Bat3.3 (Pin_3), D5.2 (A), U10.21 (VOUT), U10.22 (VOUT)
- new net GND: Bat2.1 (Pin_1), Bat3.1 (Pin_1), C10.2, C11.2, C13.2, C14.2, C19.1, C2.2, C20.1, C21.1, C22.1, C23.1, C24.2, C25.2, C26.2, C27.2, C28.1, C29.1, C3.2, C30.1, C31.1, C32.2, C33.1, C34.2, C36.2, C37.2, C38.1, C39.2, C4.2, C40.2, C41.2, C43.2, C5.2, C8.2, C9.2, D3.1 (K), D4.1 (K), D6.2 (A), J1.1 (Pin_1), J2.A1 (GND), J2.A12 (GND), J2.B1 (GND), J2.B12 (GND), J6.2 (Ext), Q1.2 (E), R34.2, R35.2, R36.2, R37.2, R41.2, R42.2, R43.2, R44.2, SW2.C, SW2.S2, SW3.1, SW4.2, U1.1 (1~{OE}), U1.15 (2~{OE}), U1.8 (GND), U10.18 (PGND), U10.24 (VBAT_GND), U11.2 (GND), U12.4 (V-), U13.2 (GND), U4.8 (GND), U5.1 (GND), U5.40 (GND), U5.41 (GND), U6.10 (SENB), U6.15 (GND), U7.10 (MD0), U7.11 (MD1), U7.12 (FMT), U7.2 (AGND), U7.5 (DGND), U8.5 (A), U9.10 (MD0), U9.11 (MD1), U9.12 (FMT), U9.2 (AGND), U9.5 (DGND)
- no-connect marks 13 -> 4
Other:
- moved on the sheet: Bat2, Bat3, J2, J7, L6

Commit message: work on rf frontend and battery charger
Parts:
- removed C33, C38, C39: 100n, Capacitor_SMD:C_0603_1608Metric, symbol uRX:C_Small
- removed SW2: RotaryEncoder_Switch, RotaryEncoder_Alps_EC11E-Switch_Vertical_H20mm, symbol Device:RotaryEncoder_Switch
- added C44, C45, C46: 100n, Capacitor_SMD:C_0603_1608Metric, symbol uRX:C_Small
- added SW1: RotaryEncoder_Switch, RotaryEncoder_Alps_EC11E-Switch_Vertical_H20mm, symbol Device:RotaryEncoder_Switch
Connections:
- net GND: now also U8.2 (A), C44.2, C45.1, C46.1, SW1.C, SW1.S2; no longer U8.5 (A)
- net Q_BAT_STAT: now also U5.25 (GPIO48/SPICLK_N/SUBSPICLK_N_DIFF); no longer U5.39 (GPIO1/TOUCH1/ADC1_CH0)
- net VRev2.5: now also U8.1 (K); no longer U8.4 (K)
- net at U5.31 (GPIO38/FSPIWP/SUBSPIWP): now also C44.1, SW1.S1
- net at U5.32 (MTCK/GPIO39/CLK_OUT3/SUBSPICS1): now also C45.2, SW1.A
- net at U5.33 (MTDO/GPIO40/CLK_OUT2): now also C46.2, SW1.B
