File: kicad/uRX/uRX.kicad_sch (KiCad schematic)
At the start: 170 parts, among them J1 RF_AM_GND, J10 GPIO_A, J11 Bat1, J12 TPH, J2 C165948, J3 Loudspeaker, J4 Display, J5 e-ink, J6 U.FL, J7 GPS, J8 Bat0, J9 RF_AM__In, Q1 BC847, Q2 BC847, Q3 BC847, SW1 RotaryEncoder_Switch, SW2 SW_DPDT_x2, SW3 Reset, SW4 Boot, U1 CBT3253, U10 IP2326, U11 LP2985-5.0, U12 OPA2211, U13 HT733333, U2 LM4562, U3 PAM8406D, U4 Si5351A-B-GT, U5 ESP32-S3-WROOM-2, U6 Si4732-A10, U7 PCM1808PWR, U8 LM4040-2.5, U9 PCM1808PWR, X1 X322525MOB4SI, Y2 32768kHz

Commit message: cleanup
Connections:
- net +3.3V: now also J12.1 (Pin_1); no longer J12.4 (Pin_4)
- net GND: now also J12.3 (Pin_3); no longer J12.2 (Pin_2)
- net SCL: now also J12.4 (Pin_4); no longer J12.1 (Pin_1)
- net SDA: now also J12.2 (Pin_2); no longer J12.3 (Pin_3)
Changed lines of the file:
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@@
 		)
 	)
-	(label "SDA"
+	(label "GND"
 		(at 27.94 147.32 0)
 		(effects
@@
 		)
 	)
-	(label "SCL"
+	(label "+3.3V"
 		(at 27.94 142.24 0)
 		(effects
@@
 		)
 	)
-	(label "GND"
+	(label "SDA"
 		(at 27.94 144.78 0)
 		(effects
@@
 		)
 	)
-	(label "+3.3V"
+	(label "SCL"
 		(at 27.94 149.86 0)
 		(effects

Commit message: add dac
Parts:
- removed C47, C48, C52: 1u, Capacitor_SMD:C_0603_1608Metric, symbol Device:C_Small
- removed C53: 10n, Capacitor_SMD:C_0603_1608Metric, symbol uRX:C_Small
- removed J10: GPIO_A, PinHeader_1x12_P2.54mm_Vertical, symbol Connector:Conn_01x12_Pin
- removed JP1: AudioMix, Connector_PinHeader_2.54mm:PinHeader_1x02_P2.54mm_Vertical, symbol Jumper:Jumper_2_Open
- removed R24, R25: 1k, Resistor_SMD:R_0603_1608Metric, symbol uRX:R
- removed R31, R32: 1k, Resistor_SMD:R_0603_1608Metric, symbol Device:R
- added C47: 4.7u, Capacitor_SMD:C_0603_1608Metric, symbol uRX:C_Small
- added C58, C59, C60: 2.2u, Capacitor_SMD:C_0603_1608Metric, symbol Device:C_Small
- added C61: 100n, Capacitor_SMD:C_0603_1608Metric, symbol Device:C_Small
- added C62: 10u, Capacitor_SMD:C_0603_1608Metric, symbol Device:C_Small
- added C63: 2.2n, Capacitor_SMD:C_0603_1608Metric, symbol Device:C_Small
- added J13: Power, PinHeader_1x04_P2.54mm_Vertical, symbol Connector:Conn_01x04_Pin
- added R50: 10k, Resistor_SMD:R_0603_1608Metric, symbol Device:R
- added R51: 470, Resistor_SMD:R_0603_1608Metric, symbol Device:R
- added R52: 22, Resistor_SMD:R_0603_1608Metric, symbol Device:R
- added U14: PCM5102A, Package_SO:TSSOP-20_4.4x6.5mm_P0.65mm, symbol Audio:PCM5102A
Connections:
- net +3.3V: now also C61.1, C62.1, J13.2 (Pin_2), R50.1, U14.1 (CPVDD), U14.20 (DVDD), U14.8 (AVDD)
- net +5V: now also J13.1 (Pin_1)
- net GND: now also C58.2, C60.2, C61.2, C62.2, C63.2, J13.3 (Pin_3), J13.4 (Pin_4), U14.10 (DEMP), U14.11 (FLT), U14.12 (SCK), U14.16 (FMT), U14.19 (DGND), U14.3 (CPGND)
- net I2S_BCK: now also U14.13 (BCK)
- net I2S_LRCK: now also U14.15 (LRCK)
- net at J3.1 (Pin_1): now also U3.1 (+OUT_L); no longer U3.16 (+OUT_R)
- net at J3.2 (Pin_2): no longer U3.14 (-OUT_R)
- net at U3.10 (INR): now also C54.2
- net at U3.7 (INL): now also C47.1; no longer C54.2
- net AUDIO_MONO_ESP: no longer names the net of U5.18 (GPIO10/TOUCH10/ADC1_CH9/FSPICS0/FSPIIO4/SUBSPICS0)
- net AUDIO_MONO_ESP: now also R52.2
- net I2S0_DOUT renamed I2S_DIN0
- net I2S1_DOUT renamed I2S_DIN1
- new net: R50.2, U14.17 (XSMT)
- new net: C60.1, U14.18 (LDOO)
- new net: C59.1, U14.2 (CAPP)
- new net: C59.2, U14.4 (CAPM)
- new net: C58.1, U14.5 (VNEG)
- new net: R51.1, U14.6 (OUTL)
- new net AGND: U14.9 (AGND)
- new net AUDIO_MONO_DAC: C47.2, C63.1, R51.2
- new net I2S_DOUT: R52.1, U14.14 (DIN)
- no-connect marks 7 -> 10
Other:
- moved on the sheet: J3

Commit message: esp verify code compiled
Parts:
- added NT3: NetTie_3, NetTie:NetTie-2_SMD_Pad0.5mm, symbol Device:NetTie_2
Connections:
- net GND: now also NT3.2
- net AGND: no longer names the net of U14.9 (AGND)
- net AGND: now also NT3.1
Other:
- moved on the sheet: C32, C34, C35, C36, C37, C39, C47, C49, C50, C51, C54, C55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

Commit message: cleanup
Connections:
- net L_4732: now reaches U6.1 (LOut)
- net L_4732: now also C17.1; no longer C18.1
- net R_4732: now reaches U6.16 (ROut)
- net R_4732: now also C18.1; no longer C17.1
Other:
- note added: "D/A converter"
- moved on the sheet: R17, R5, R7

Commit message: set gnd/vcc lines propperly
Parts:
- added C48: 2.2u, Capacitor_SMD:C_0603_1608Metric, symbol Device:C_Small
- added C52: 100n, Capacitor_SMD:C_0603_1608Metric, symbol Device:C_Small
- added L9: Ferrite_perl, Inductor_SMD:L_0603_1608Metric, symbol Device:L_Ferrite_Small
- C13: value 100n -> 2.2u
Connections:
- net +3.3V: now also L9.1
- net +3.3VfilteredM: no longer R5.1, U6.14 (VDD)
- net +5VfilteredQ: now also C48.1, C52.1
- net GND: now also C48.2, C52.2
- net at J3.2 (Pin_2): now also U3.3 (-OUT_L)
- new net +3.3VfilteredQ: L9.2, R5.1, U6.14 (VDD)
Other:
- moved on the sheet: C10, C11, R20
