File: kicad/uRX/_autosave-uRX.kicad_sch (KiCad schematic)
At the start: 138 parts, among them J1 RF_AM_GND, J10 GPIO_A, J11 +3.3Vfiltered, J2 C165948, J3 AudioJack2_Ground, J4 +5Vfiltered, J5 +5V, J6 U.FL, J7 +3.3Vfiltered, J8 +5Vfiltered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

Commit message: connect all together, v0
Parts:
- removed 3.3V1: +3.3V, TestPoint_THTPad_1.0x1.0mm_Drill0.5mm, symbol Connector:TestPoint
- removed 5V1: +5V, TestPoint_THTPad_1.0x1.0mm_Drill0.5mm, symbol Connector:TestPoint
- removed VBatt1: VBatt, TestPoint_THTPad_1.0x1.0mm_Drill0.5mm, symbol Connector:TestPoint
