File: kicad/uRX.old/uRX.kicad_pcb (KiCad board)
At the start: 2 copper layers, 13 x 1.4 mm, 154 parts, among them J1 RF_AM_GND, J2 C165948, J3 AudioJack2_Ground, J4 +5Vfiltered, J5 +5V, J5 Bat, J5 GND, J6 U.FL, J7 +3.3Vfiltered, J8 U.FL, J9 RF_AM__In, Q1 BC847, SW1 RotaryEncoder_Switch, SW2 SW_DPDT_x2, SW3 Reset, SW4 Boot, SW5 SW_DPDT_x2, U1 CBT3253, U10 IP2326, U11 LP2985-5.0, U12 OPA2211, U13 HT733333, U2 LM4562, U4 Si5351A-B-GT, U5 ESP32-S3-WROOM-2, U6 Si4732-A10, U7 PCM1808PWR, U8 LM4040-2.5, U9 PCM1808PWR, Y1 25MHz, Y2 32768kHz

Commit message: seafile corruption
Parts:
- removed Bat2, Bat3: JST-XH, Connector_JST:JST_XH_B3B-XH-A_1x03_P2.50mm_Vertical
- removed the C1 at (190.2, 46.2)
- removed the C2 at (254.5, 68.9)
- removed the C2 at (212.9, 88.4)
- removed the C3 at (254.5, 71.4)
- removed the C3 at (222.7, 88.4)
- removed the C4 at (254.5, 73.9)
- removed the C4 at (216.2, 88.4)
- removed the C41 at (258.5, 66.4)
- removed the C41 at (220.4, 72.1)
- removed the C43 at (220.4, 70.4)
- removed the C43 at (258.5, 68.9)
- removed the C5 at (254.5, 76.4)
- removed the C5 at (219.4, 88.4)
- removed the C8 at (221.4, 47.4)
- removed Display: , Connector_PinHeader_2.54mm:PinHeader_1x09_P2.54mm_Vertical
- removed J5 (x2): +5V, Connector_Pin:Pin_D0.9mm_L10.0mm_W2.4mm_FlatFork
- removed J5: GND, Connector_Pin:Pin_D0.9mm_L10.0mm_W2.4mm_FlatFork
- removed J5: Bat, Connector_Pin:Pin_D0.9mm_L10.0mm_W2.4mm_FlatFork
- removed J7: +3.3Vfiltered, Connector_Pin:Pin_D0.9mm_L10.0mm_W2.4mm_FlatFork
- removed the R11 at (258.5, 71.4)
- removed the R11 at (214.6, 89.1)
- removed the R26 at (258.5, 73.9)
- removed the R26 at (220.7, 58.9)
- removed the R27 at (258.5, 76.4)
- removed the R27 at (216.4, 74.6)
- removed the R28 at (258.5, 78.9)
- removed the R28 at (222.2, 68.1)
- removed Rf2, Rf3: 47, Resistor_SMD:R_0603_1608Metric
- removed the Rf6 at (217.2, 71.1)
- removed the Rf6 at (262.5, 66.4)
- removed the Rf7 at (222.2, 64.6)
- removed the Rf7 at (262.5, 68.9)
- removed the Rg1 at (262.5, 71.4)
- removed the Rg1 at (216.2, 58.9)
- removed the Rg2 at (262.5, 73.9)
- removed the Rg2 at (218.5, 58.9)
- removed SW5: SW_DPDT_x2, Button_Switch_THT:SW_E-Switch_EG1224_SPDT_Angled
- removed the U2 at (218.4, 99.6)
- removed Y1: 25MHz, Crystal:Crystal_SMD_3225-4Pin_3.2x2.5mm
- added 2211Out1: TestPoint, TestPoint:TestPoint_THTPad_1.0x1.0mm_Drill0.5mm, F.Cu at (205.0, 66.3)
- added C2: 220n, Capacitor_SMD:C_0603_1608Metric, F.Cu at (216.2, 70.0)
- added C3: 220n, Capacitor_SMD:C_0603_1608Metric, F.Cu at (216.2, 79.2)
- added C33: 10n, Capacitor_SMD:C_0603_1608Metric, F.Cu at (184.0, 75.0)
- added C38: 10n, Capacitor_SMD:C_0603_1608Metric, F.Cu at (184.0, 73.3)
- added C39: 1u, Capacitor_SMD:C_0603_1608Metric, F.Cu at (136.8, 91.2)
- added C4: 220n, Capacitor_SMD:C_0603_1608Metric, F.Cu at (216.2, 73.0)
- added C41: 2.2u, Capacitor_SMD:C_0603_1608Metric, F.Cu at (221.0, 64.8)
- added C43: 100n, Capacitor_SMD:C_0603_1608Metric, F.Cu at (222.8, 62.8)
- added C47: 1u, Capacitor_SMD:C_0603_1608Metric, F.Cu at (176.4, 66.0)
- added C48: 1u, Capacitor_SMD:C_0603_1608Metric, F.Cu at (184.8, 66.0)
- added C49: 10u, Capacitor_SMD:C_0603_1608Metric, F.Cu at (152.5, 79.8)
- added C5: 220n, Capacitor_SMD:C_0603_1608Metric, F.Cu at (216.2, 76.2)
- added C50: 100n, Capacitor_SMD:C_0603_1608Metric, F.Cu at (152.5, 82.0)
- added C51: 100n, Capacitor_SMD:C_0603_1608Metric, F.Cu at (136.8, 87.8)
- added C52: 1u, Capacitor_SMD:C_0603_1608Metric, F.Cu at (154.5, 89.2)
- added C53: 10n, Capacitor_SMD:C_0603_1608Metric, F.Cu at (147.0, 91.8)
- added C54: 1u, Capacitor_SMD:C_0603_1608Metric, F.Cu at (136.8, 89.5)
- added C55: 10u, Capacitor_SMD:C_0805_2012Metric, F.Cu at (135.1, 127.2)
- added C56: 10u, Capacitor_SMD:C_0805_2012Metric, F.Cu at (124.8, 115.0)
- added C57: 10u, Capacitor_SMD:C_0805_2012Metric, F.Cu at (121.0, 114.0)
- added J10: GPIO_A, Connector_PinHeader_2.54mm:PinHeader_1x12_P2.54mm_Vertical, F.Cu at (130.0, 108.2)
- added J11: Bat1, Connector_JST:JST_PH_B2B-PH-K_1x02_P2.00mm_Vertical, F.Cu at (82.2, 98.0)
- added L1: Ferrite_perl, Inductor_SMD:L_0603_1608Metric, F.Cu at (126.0, 82.8)
- added L3: Ferrite_perl, Inductor_SMD:L_0603_1608Metric, F.Cu at (125.0, 80.2)
- added M2: , MountingHole:MountingHole_2.2mm_M2_DIN965, F.Cu at (139.3, 68.4)
- added NT1: NetTie_2, NetTie:NetTie-2_SMD_Pad0.5mm, F.Cu at (196.7, 56.7)
- added NT2: NetTie_2, NetTie:NetTie-2_SMD_Pad0.5mm, F.Cu at (196.7, 59.3)
- added R11: 1k, Resistor_SMD:R_0603_1608Metric, F.Cu at (217.1, 71.5)
- added R17: 22, Resistor_SMD:R_0603_1608Metric, F.Cu at (186.1, 97.8)
- added R21: 10k, Resistor_SMD:R_0603_1608Metric, F.Cu at (99.8, 100.2)
- added R22: 10k, Resistor_SMD:R_0603_1608Metric, F.Cu at (94.2, 100.2)
- added R23: 10, Resistor_SMD:R_0603_1608Metric, F.Cu at (136.8, 86.0)
- added R24: 1k, Resistor_SMD:R_0603_1608Metric, F.Cu at (157.2, 90.0)
- added R26: 100k, Resistor_SMD:R_0603_1608Metric, F.Cu at (218.1, 52.0)
- added R27: 22, Resistor_SMD:R_0603_1608Metric, F.Cu at (216.2, 68.2)
- added R28: 22, Resistor_SMD:R_0603_1608Metric, F.Cu at (214.7, 58.3)
- added R31: 1k, Resistor_SMD:R_0603_1608Metric, F.Cu at (171.8, 66.0)
- added R32: 1k, Resistor_SMD:R_0603_1608Metric, F.Cu at (171.7, 69.0)
- added R7: 22, Resistor_SMD:R_0603_1608Metric, F.Cu at (168.2, 87.7)
- added Rf4: 47, Resistor_SMD:R_0603_1608Metric, F.Cu at (201.0, 75.0)
- added Rf5: 47, Resistor_SMD:R_0603_1608Metric, F.Cu at (204.0, 73.2)
- added Rf6: 604, Resistor_SMD:R_0603_1608Metric, F.Cu at (218.0, 66.0)
- added Rf7: 604, Resistor_SMD:R_0603_1608Metric, F.Cu at (217.3, 54.5)
- added Rf8: 47, Resistor_SMD:R_0603_1608Metric, F.Cu at (181.7, 80.3)
- added Rg1: 604, Resistor_SMD:R_0603_1608Metric, F.Cu at (213.6, 52.0)
- added Rg2: 604, Resistor_SMD:R_0603_1608Metric, F.Cu at (215.9, 52.0)
- added TP4: CLK0, TestPoint:TestPoint_THTPad_1.0x1.0mm_Drill0.5mm, F.Cu at (190.0, 78.0)
- added TP5: CLK1, TestPoint:TestPoint_THTPad_1.0x1.0mm_Drill0.5mm, F.Cu at (190.0, 70.5)
- added TP6: CLK2, TestPoint:TestPoint_THTPad_1.0x1.0mm_Drill0.5mm, F.Cu at (186.9, 80.3)
- added U3: PAM8406D, Package_SO:SOIC-16_3.9x9.9mm_P1.27mm, F.Cu at (144.5, 85.2)
- added VRef1: VRef, TestPoint:TestPoint_THTPad_1.0x1.0mm_Drill0.5mm, F.Cu at (221.8, 89.0)
- added X1: X322525MOB4SI, Crystal:Crystal_SMD_3225-4Pin_3.2x2.5mm, F.Cu at (172.7, 74.8)
- C13, C14: value 2..20p -> 100n
- C17, C18: value 4.7u -> 1u
- C34: footprint Capacitor_SMD:C_0603_1608Metric -> Capacitor_SMD:C_0805_2012Metric
- J3: value AudioJack2_Ground -> Loudspeaker; footprint Connector_Audio:Jack_3.5mm_CUI_SJ1-3523N_Horizontal -> Connector_JST:JST_PH_B2B-PH-K_1x02_P2.00mm_Vertical
- J4: value +5Vfiltered -> Display; footprint Connector_Pin:Pin_D0.9mm_L10.0mm_W2.4mm_FlatFork -> Connector_PinHeader_2.54mm:PinHeader_1x08_P2.54mm_Vertical
- J8: value U.FL -> Bat0; footprint Connector_Coaxial:SMA_Molex_73251-1153_EdgeMount_Horizontal -> Connector_JST:JST_PH_B2B-PH-K_1x02_P2.00mm_Vertical
- L5, L6: value Ferrite_perl -> L_Core_Ferrite; footprint Inductor_SMD:L_0603_1608Metric -> Inductor_SMD:L_Taiyo-Yuden_NR-40xx
- R16: value 22 -> 10k
- R25: value 22 -> 1k
- Rf1: value 33 -> 47
- SW1: moved to B.Cu
- SW2: footprint Button_Switch_THT:SW_E-Switch_EG1224_SPDT_Angled -> Button_Switch_SMD:SW_SPDT_PCM12
- moved J8 145.4 mm to (82.2, 90.0), turned to 90 degrees
- moved R5 105.0 mm to (107.8, 109.7), turned to -90 degrees
- moved J3 78.3 mm to (129.6, 74.0), turned to -90 degrees
- moved M2 66.8 mm to (21.5, 69.2)
- moved C18 64.3 mm to (188.5, 66.0)
- moved M2 62.2 mm to (22.0, 87.8)
- moved C17 58.5 mm to (180.4, 66.0)
- moved M2 57.9 mm to (139.1, 48.1)
- moved U2 57.2 mm to (215.9, 90.5), turned to 90 degrees
- moved C10 56.3 mm to (223.0, 68.2), turned to -90 degrees
- moved C1 54.5 mm to (201.2, 54.6), turned to 90 degrees
- moved R18 50.5 mm to (220.8, 86.2)
- moved C11 49.2 mm to (221.0, 68.2), turned to -90 degrees
- moved J4 47.9 mm to (82.8, 67.3), turned to 180 degrees
- moved R25 47.6 mm to (151.0, 89.2), turned to 0 degrees
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Connections:
- C13 pad 1: Net-(U4-XA) -> +3.3V
- C14 pad 1: Net-(U4-XB) -> +3.3V
- C17 pad 1: Net-(U9-VINR) -> Net-(U6-ROut)
- C17 pad 2: Net-(U6-LOut) -> Net-(U9-VINL)
- C18 pad 1: Net-(U9-VINL) -> Net-(U6-LOut)
- C18 pad 2: Net-(U6-ROut) -> Net-(U9-VINR)
- C29 pad 2: +5Vfiltered -> +5V
- C30 pad 2: +3.3Vfiltered -> +3.3V
- C31 pad 2: +5Vfiltered -> +5V
- C34 pad 1: VBUS -> VBUSfiltered
- C40 pad 1: Net-(SW5A-C) -> Net-(D6-K)
- C45 pad 2: Net-(U5-MTCK/GPIO39/CLK_OUT3/SUBSPICS1) -> Net-(U5-MTDO/GPIO40/CLK_OUT2)
- C46 pad 2: Net-(U5-MTDO/GPIO40/CLK_OUT2) -> Net-(U5-MTCK/GPIO39/CLK_OUT3/SUBSPICS1)
- D2 pad 2: VBUS -> VBUSfiltered
- J2 pad A4: VBUS -> Net-(C55-Pad2)
- J2 pad A9: VBUS -> Net-(C55-Pad2)
- J2 pad B4: VBUS -> Net-(C55-Pad2)
- J2 pad B9: VBUS -> Net-(C55-Pad2)
- J4 pad 1: Net-(J4-Pin_1) -> GND
- J8 pad 1: Net-(J8-In) -> Net-(J11-Pin_2)
- J8 pad 2: GND -> +VBatt
- L2 pad 2: VBUS -> VBUSfiltered
- L4 pad 1: Net-(SW5A-C) -> Net-(D6-K)
- L5 pad 1: +3.3V -> VBUSfiltered
- L5 pad 2: Net-(J7-Pin_1) -> Net-(C55-Pad2)
- L6 pad 1: +5V -> +VBatt
- L6 pad 2: Net-(J4-Pin_1) -> Net-(C56-Pad2)
- R16 pad 1: /I2S0_DOUT -> +3.3V
- R16 pad 2: Net-(U5-GPIO13/TOUCH13/ADC2_CH2/FSPIQ/FSPIIO7/SUBSPIQ) -> Net-(U5-GPIO38/FSPIWP/SUBSPIWP)
- R25 pad 1: /I2S1_DOUT -> /AUDIO_MONO_4732
- R25 pad 2: Net-(U5-GPIO14/TOUCH14/ADC2_CH3/FSPIWP/FSPIDQS/SUBSPIWP) -> Net-(C52-Pad2)
- R39 pad 2: Net-(Bat2-Pin_2) -> Net-(J11-Pin_2)
- R44 pad 1: VBUS -> VBUSfiltered
- R5 pad 1: +3.3Vfiltered -> +3.3V
- Rf1 pad 1: ADC_SCKI -> Net-(U4-CLK2)
- Rf1 pad 2: Net-(U4-CLK2) -> ADC1_SCKI
- SW2 pad 1: Net-(SW2A-A) -> unconnected-(SW2A-A-Pad1)
- SW2 pad 3: unconnected-(SW2A-C-Pad3) -> Net-(SW2A-C)
- U10 pad 1: unconnected-(U10-DM-Pad1) -> USB_D-
- U10 pad 12: VBUS -> VBUSfiltered
- U10 pad 13: VBUS -> VBUSfiltered
- U10 pad 15: Net-(U10-LX-Pad15) -> Net-(C35-Pad1)
- U10 pad 17: Net-(U10-LX-Pad15) -> Net-(C35-Pad1)
- U10 pad 2: unconnected-(U10-DP-Pad2) -> USB_D+
- U10 pad 21: +VBatt -> Net-(C56-Pad2)
- U10 pad 22: +VBatt -> Net-(C56-Pad2)
- U11 pad 5: Net-(SW2A-A) -> Net-(SW2A-C)
- U2 pad 4: (no net) -> GND
- U2 pad 8: (no net) -> +5Vfiltered
- U5 pad 18: ADC_SCKI -> /AUDIO_MONO_ESP
- U5 pad 21: Net-(U5-GPIO13/TOUCH13/ADC2_CH2/FSPIQ/FSPIIO7/SUBSPIQ) -> /I2S0_DOUT
- U5 pad 22: Net-(U5-GPIO14/TOUCH14/ADC2_CH3/FSPIWP/FSPIDQS/SUBSPIWP) -> /I2S1_DOUT
- U5 pad 23: unconnected-(U5-GPIO21-Pad23) -> RST_4732
- U5 pad 24: unconnected-(U5-GPIO47/SPICLK_P/SUBSPICLK_P_DIFF-Pad24) -> Q_BAT_STAT
- U5 pad 25: Q_BAT_STAT -> /AUDIO_SHND
- U5 pad 26: unconnected-(U5-GPIO45-Pad26) -> /AUDIO_MUTE
- U5 pad 34: unconnected-(U5-MTDI/GPIO41/CLK_OUT1-Pad34) -> /D_BLK
- U5 pad 35: unconnected-(U5-MTMS/GPIO42-Pad35) -> /D_CS
- U5 pad 36: unconnected-(U5-U0RXD/GPIO44/CLK_OUT2-Pad36) -> /D_DC
- U5 pad 37: unconnected-(U5-U0TXD/GPIO43/CLK_OUT1-Pad37) -> /D_RES
- U5 pad 7: RST_4732 -> unconnected-(U5-GPIO7/TOUCH7/ADC1_CH6-Pad7)
- U6 pad 14: +3.3Vfiltered -> +3.3V
- U6 pad 7: Earth -> Net-(U6-RFGND)
- U7 pad 6: ADC_SCKI -> ADC0_SCKI
- U7 pad 9: /I2S0_DOUT -> Net-(U7-DOUT)
- U9 pad 1: +5Vfiltered -> +5V
- U9 pad 3: +5Vfiltered -> +5V
- U9 pad 4: +3.3Vfiltered -> +3.3V
- U9 pad 6: ADC_SCKI -> ADC1_SCKI
- U9 pad 9: /I2S1_DOUT -> Net-(U9-DOUT)
Routing:
- net GND: track 166.1 -> 529.3 mm, vias 12 -> 154
- net /SDA: track 2.63 -> 157.0 mm, vias 0 -> 9
- net /SCL: track 5.83 -> 152.7 mm, vias 0 -> 9
- net /I2S_BCK: track 0.00 -> 141.1 mm, vias 0 -> 3
- net RST_4732: track 0.00 -> 131.4 mm, vias 0 -> 3
- net /I2S0_DOUT: track 0.00 -> 94.1 mm, vias 0 -> 2
- net /I2S_LRCK: track 0.00 -> 87.4 mm, vias 0 -> 1
- net /I2S1_DOUT: track 0.00 -> 78.0 mm, vias 0 -> 1
- net /AUDIO_MONO_ESP: track 0.00 -> 72.2 mm, vias 0 -> 4
- net /D_BLK: track 0.00 -> 66.5 mm, vias 0 -> 1
- net /VRev2.5: track 15.7 -> 79.3 mm
- net /D_CS: track 0.00 -> 63.5 mm, vias 0 -> 1
- net /D_DC: track 0.00 -> 60.4 mm, vias 0 -> 1
- net Net-(J11-Pin_2): track 0.00 -> 60.0 mm
- net /AUDIO_SHND: track 0.00 -> 59.9 mm, vias 0 -> 2
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Other:
- board outline removed
