File: kicad/uRX.old/uRX.kicad_sch (KiCad schematic)
At the start: 133 parts, among them J1 RF_AM_GND, J10 GPIO_A, J2 C165948, J3 AudioJack2_Ground, J4 Display, J6 U.FL, J9 RF_AM__In, Q1 BC847, SW1 RotaryEncoder_Switch, SW2 SW_DPDT_x2, SW3 Reset, SW4 Boot, U1 CBT3253, U10 IP2326, U11 LP2985-5.0, U12 OPA2211, U13 HT733333, U2 LM4562, U4 Si5351A-B-GT, U5 ESP32-S3-WROOM-2, U6 Si4732-A10, U7 PCM1808PWR, U8 LM4040-2.5, U9 PCM1808PWR, X1 X322525MOB4SI, Y2 32768kHz

Commit message: pcb digital zone
Parts:
- removed J4: Display, PinHeader_1x08_P2.54mm_Vertical, symbol Connector:Conn_01x08_Pin
- removed L1, L3: Ferrite_perl, Inductor_SMD:L_0603_1608Metric, symbol Device:L_Ferrite_Small
- removed R16, R21, R22: 10k, Resistor_SMD:R_0603_1608Metric, symbol Device:R_Small
- removed R17, R7: 22, Resistor_SMD:R_0603_1608Metric, symbol Device:R
- added GND1: TestPoint_2Pole, TestPoint_2Pads_Pitch2.54mm_Drill0.8mm, symbol Connector:TestPoint_2Pole
- added J11, J7: +3.3Vfiltered, Connector_Pin:Pin_D0.9mm_L10.0mm_W2.4mm_FlatFork, symbol Connector_Generic:Conn_01x01
- added J4, J8: +5Vfiltered, Connector_Pin:Pin_D0.9mm_L10.0mm_W2.4mm_FlatFork, symbol Connector_Generic:Conn_01x01
- added J5: +5V, Connector_Pin:Pin_D0.9mm_L10.0mm_W2.4mm_FlatFork, symbol Connector_Generic:Conn_01x01
- added L5, L6: Ferrite_perl, Inductor_SMD:L_0603_1608Metric, symbol Device:L_Ferrite_Small
- added R16, R25: 22, Resistor_SMD:R_0603_1608Metric, symbol Device:R
- SW2: footprint Button_Switch_SMD:SW_SPDT_PCM12 -> SW_E-Switch_EG1224_SPDT_Angled
Connections:
- net +3.3V: now also L5.1
- net +3.3Vfiltered: no longer J10.11 (Pin_11)
- net +5V: now also L6.1
- net +5Vfiltered: no longer J10.12 (Pin_12)
- net GND: now also GND1.1, GND1.2
- net I2S0_DOUT: now also U7.9 (DOUT), R16.1; no longer U5.21 (GPIO13/TOUCH13/ADC2_CH2/FSPIQ/FSPIIO7/SUBSPIQ)
- net I2S1_DOUT: now also U9.9 (DOUT), R25.1; no longer U5.22 (GPIO14/TOUCH14/ADC2_CH3/FSPIWP/FSPIDQS/SUBSPIWP)
- net D_BLK: no longer names the net of U5.34 (MTDI/GPIO41/CLK_OUT1)
- net D_CS: no longer names the net of U5.35 (MTMS/GPIO42)
- net D_DC: no longer names the net of U5.36 (U0RXD/GPIO44/CLK_OUT2)
- net D_RES: no longer names the net of U5.37 (U0TXD/GPIO43/CLK_OUT1)
- new net: J7.1 (Pin_1), L5.2
- new net: R16.2, U5.21 (GPIO13/TOUCH13/ADC2_CH2/FSPIQ/FSPIIO7/SUBSPIQ)
- new net: J4.1 (Pin_1), L6.2
- new net: R25.2, U5.22 (GPIO14/TOUCH14/ADC2_CH3/FSPIWP/FSPIDQS/SUBSPIWP)
- new net: J10.11 (Pin_11), J11.1 (Pin_1)
- new net: J10.12 (Pin_12), J8.1 (Pin_1)
Other:
- moved on the sheet: R13, R15, R9

Commit message: seafile corruption
Parts:
- removed Bat2, Bat3: JST-XH, Connector_JST:JST_XH_B3B-XH-A_1x03_P2.50mm_Vertical, symbol uRX:Conn_01x03
- removed GND1: TestPoint_2Pole, TestPoint_2Pads_Pitch2.54mm_Drill0.8mm, symbol Connector:TestPoint_2Pole
- removed J11, J7: +3.3Vfiltered, Connector_Pin:Pin_D0.9mm_L10.0mm_W2.4mm_FlatFork, symbol Connector_Generic:Conn_01x01
- removed J3: AudioJack2_Ground, Connector_Audio:Jack_3.5mm_CUI_SJ1-3523N_Horizontal, symbol Connector_Audio:AudioJack2_Ground
- removed J4, J8: +5Vfiltered, Connector_Pin:Pin_D0.9mm_L10.0mm_W2.4mm_FlatFork, symbol Connector_Generic:Conn_01x01
- removed J5: +5V, Connector_Pin:Pin_D0.9mm_L10.0mm_W2.4mm_FlatFork, symbol Connector_Generic:Conn_01x01
- removed R16, R25: 22, Resistor_SMD:R_0603_1608Metric, symbol Device:R
- added C39, C54: 1u, Capacitor_SMD:C_0603_1608Metric, symbol uRX:C_Small
- added C47, C48, C52: 1u, Capacitor_SMD:C_0603_1608Metric, symbol Device:C_Small
- added C49: 10u, Capacitor_SMD:C_0603_1608Metric, symbol uRX:C_Small
- added C50, C51: 100n, Capacitor_SMD:C_0603_1608Metric, symbol uRX:C_Small
- added C53: 10n, Capacitor_SMD:C_0603_1608Metric, symbol uRX:C_Small
- added C55, C56, C57: 10u, C_0805_2012Metric, symbol uRX:C_Small
- added J11: Bat1, Connector_JST:JST_PH_B2B-PH-K_1x02_P2.00mm_Vertical, symbol Connector_Generic:Conn_01x02
- added J3: Loudspeaker, Connector_JST:JST_PH_B2B-PH-K_1x02_P2.00mm_Vertical, symbol Connector_Generic:Conn_01x02
- added J4: Display, PinHeader_1x08_P2.54mm_Vertical, symbol Connector:Conn_01x08_Pin
- added J8: Bat0, Connector_JST:JST_PH_B2B-PH-K_1x02_P2.00mm_Vertical, symbol Connector_Generic:Conn_01x02
- added L1, L3: Ferrite_perl, Inductor_SMD:L_0603_1608Metric, symbol Device:L_Ferrite_Small
- added NT1, NT2: NetTie_2, NetTie:NetTie-2_SMD_Pad0.5mm, symbol Device:NetTie_2
- added R16, R21, R22: 10k, Resistor_SMD:R_0603_1608Metric, symbol Device:R_Small
- added R17, R7: 22, Resistor_SMD:R_0603_1608Metric, symbol Device:R
- added R23: 10, Resistor_SMD:R_0603_1608Metric, symbol uRX:R
- added R24, R25: 1k, Resistor_SMD:R_0603_1608Metric, symbol uRX:R
- added R31, R32: 1k, Resistor_SMD:R_0603_1608Metric, symbol Device:R
- added Rf8: 47, Resistor_SMD:R_0603_1608Metric, symbol Device:R
- added unit 3 of U2
- added U3: PAM8406D, Package_SO:SOIC-16_3.9x9.9mm_P1.27mm, symbol Amplifier_Audio:PAM8406D
- C17, C18: value 4.7u -> 1u
- C34: footprint Capacitor_SMD:C_0603_1608Metric -> C_0805_2012Metric
- L5, L6: value Ferrite_perl -> L_Core_Ferrite; footprint Inductor_SMD:L_0603_1608Metric -> Inductor_SMD:L_Taiyo-Yuden_NR-40xx
- SW2: footprint SW_E-Switch_EG1224_SPDT_Angled -> Button_Switch_SMD:SW_SPDT_PCM12
Connections:
- net +3.3V: now also C49.2, C50.2, J4.2 (Pin_2), L1.1, R16.1, R21.1, R22.1, R23.1, U3.13 (PVDDR), U3.4 (PVDDL), U3.9 (MODE); no longer L5.1
- net +3.3Vfiltered: now also J10.11 (Pin_11), L1.2
- net +5V: now also L3.1; no longer L6.1
- net +5Vfiltered: now also J10.12 (Pin_12), L3.2, U2.8 (V+)
- net +VBatt: now also L6.1, C57.2, J8.2 (Pin_2); no longer U10.21 (VOUT), U10.22 (VOUT)
- net Earth: now also NT1.1; no longer U6.7 (RFGND)
- net GND: now also C39.1, C49.1, C50.1, C51.1, C53.1, C54.1, C55.1, C56.1, C57.1, J11.1 (Pin_1), J4.1 (Pin_1), NT1.2, NT2.2, U2.4 (V-), U3.11 (GND), U3.15 (PGNDR), U3.2 (PGNDL)
- net I2S0_DOUT: now also U5.21 (GPIO13/TOUCH13/ADC2_CH2/FSPIQ/FSPIIO7/SUBSPIQ), R17.2; no longer U7.9 (DOUT)
- net I2S1_DOUT: now also U5.22 (GPIO14/TOUCH14/ADC2_CH3/FSPIWP/FSPIDQS/SUBSPIWP), R7.2; no longer U9.9 (DOUT)
- net Q_BAT_STAT: now also U5.24 (GPIO47/SPICLK_P/SUBSPICLK_P_DIFF); no longer U5.25 (GPIO48/SPICLK_N/SUBSPICLK_N_DIFF)
- net SCL: now also J4.3 (Pin_3)
- net SDA: now also J4.4 (Pin_4)
- net USB_D+: now also U10.2 (DP)
- net USB_D-: now also U10.1 (DM)
- net at SW2.1 (A): no longer U11.5 (VOUT)
- net at SW2.3 (C): now also U11.5 (VOUT)
- net at L5.2: now also J2.A4 (VBUS), J2.A9 (VBUS), J2.B4 (VBUS), J2.B9 (VBUS), C55.2
- net at SW1.A, U5.32 (MTCK/GPIO39/CLK_OUT3/SUBSPICS1): now also C46.2, R21.2; no longer C45.2
- net at SW1.B, U5.33 (MTDO/GPIO40/CLK_OUT2): now also C45.2, R22.2; no longer C46.2
- net at C44.1, SW1.S1, U5.31 (GPIO38/FSPIWP/SUBSPIWP): now also R16.2
- net at R39.2: now also J11.2 (Pin_2), J8.1 (Pin_1)
- net at L6.2: now also U10.21 (VOUT), U10.22 (VOUT), C56.2
- net at U6.1 (LOut): now also C18.1, C48.2; no longer C17.2
- net at U6.16 (ROut): now also C17.1, C47.2; no longer C18.2
- net at U4.6 (CLK2): now also Rf1.1, TP6.1, Rf8.1; no longer Rf1.2
- net at U9.14 (VINR): now also C18.2; no longer C17.1
- net AUDIO_MUTE: now reaches U5.26 (GPIO45)
- net AUDIO_MUTE: now also U3.5 (~{MUTE})
- net D_BLK: now reaches U5.34 (MTDI/GPIO41/CLK_OUT1)
- net D_BLK: now also J4.8 (Pin_8)
- net D_CS: now reaches U5.35 (MTMS/GPIO42)
- net D_CS: now also J4.7 (Pin_7)
- net D_DC: now reaches U5.36 (U0RXD/GPIO44/CLK_OUT2)
- net D_DC: now also J4.6 (Pin_6)
- net D_RES: now reaches U5.37 (U0TXD/GPIO43/CLK_OUT1)
- net D_RES: now also J4.5 (Pin_5)
- net at U9.13 (VINL): now also C17.2; no longer C18.1
- removed net ADC_SCKI: J10.3 (Pin_3), Rf1.1, TP6.1, U5.18 (GPIO10/TOUCH10/ADC1_CH9/FSPICS0/FSPIIO4/SUBSPICS0), U7.6 (SCKI), U9.6 (SCKI)
- net VBUS renamed VBUSfiltered
- net VBUSfiltered: now also L5.1; no longer J2.A4 (VBUS), J2.A9 (VBUS), J2.B4 (VBUS), J2.B9 (VBUS)
- new net: NT2.1, U6.7 (RFGND)
- new net: J3.1 (Pin_1), U3.1 (+OUT_L)
- new net: J3.2 (Pin_2), U3.3 (-OUT_L)
- new net: C52.2, R25.2
- new net: R7.1, U9.9 (DOUT)
- new net: C51.2, R23.2, U3.6 (VDD)
- new net: C52.1, C53.2, R24.1
- new net: C39.2, U3.8 (VREF)
- new net: C47.1, R31.2
- new net: R17.1, U7.9 (DOUT)
- new net: C54.2, U3.7 (INL)
- new net: C48.1, R32.2
- new net ADC0_SCKI: Rf8.2, U7.6 (SCKI)
- new net ADC1_SCKI: Rf1.2, U9.6 (SCKI)
- new net AUDIO_MONO_4732: R25.1, R31.1, R32.1, U3.10 (INR)
- new net AUDIO_MONO_ESP: J10.3 (Pin_3), R24.2, U5.18 (GPIO10/TOUCH10/ADC1_CH9/FSPICS0/FSPIIO4/SUBSPICS0)
- new net AUDIO_SHND: U3.12 (~{SHND}), U5.25 (GPIO48/SPICLK_N/SUBSPICLK_N_DIFF)
- no-connect marks 4 -> 18
Other:
- moved on the sheet: C10, C11, C17, C18, D5, R13, R15, R9
